File: Turing Machine.kicad_pcb (KiCad board)
At the start: 6 copper layers, 277 x 132 mm, 255 parts, among them J1 Conn_01x02_Socket, J10 Conn_01x02_Socket, J100 Conn_01x02_Socket, J101 Conn_01x02_Socket, J102 Conn_01x02_Socket, J103 Conn_01x02_Socket, J104 Conn_01x02_Socket, J105 Conn_01x02_Socket, J106 Conn_01x02_Socket, J107 Conn_01x02_Socket, J108 Conn_01x02_Socket, J109 Conn_01x02_Socket, J11 Conn_01x02_Socket, J110 Conn_01x02_Socket, J111 Conn_01x02_Socket, J112 Conn_01x02_Socket, J113 Conn_01x02_Socket, J114 Conn_01x02_Socket, J115 Conn_01x02_Socket, J116 Conn_01x02_Socket, J117 Conn_01x02_Socket, J118 Conn_01x02_Socket, J119 Conn_01x02_Socket, J12 Conn_01x02_Socket, J120 Conn_01x02_Socket, J121 Conn_01x02_Socket, J122 Conn_01x02_Socket, J123 Conn_01x02_Socket, J124 Conn_01x02_Socket, J125 Conn_01x02_Socket, J126 Conn_01x02_Socket, J127 Conn_01x02_Socket, J128 Conn_01x02_Socket, J129 Conn_01x02_Socket, J13 Conn_01x02_Socket, J130 Conn_01x02_Socket, J131 Conn_01x02_Socket, J132 Conn_01x02_Socket, J133 Conn_01x02_Socket, J134 Conn_01x02_Socket, J135 Conn_01x02_Socket, J136 Conn_01x02_Socket, J137 Conn_01x02_Socket, J138 Conn_01x02_Socket, J139 Conn_01x02_Socket, J14 Conn_01x02_Socket, J140 Conn_01x02_Socket, J141 Conn_01x02_Socket, J142 Conn_01x02_Socket, J143 Conn_01x02_Socket, J144 Conn_01x02_Socket, J145 Conn_01x02_Socket, J146 Conn_01x02_Socket, J147 Conn_01x02_Socket, J148 Conn_01x02_Socket, J149 Conn_01x02_Socket, J15 Conn_01x02_Socket, J150 Conn_01x02_Socket, J151 Conn_01x02_Socket, J152 Conn_01x02_Socket, J153 Conn_01x02_Socket, J154 Conn_01x02_Socket, J155 Conn_01x02_Socket, J156 Conn_01x02_Socket, J157 Conn_01x02_Socket, J158 Conn_01x02_Socket, J159 Conn_01x02_Socket, J16 Conn_01x02_Socket, J160 Conn_01x02_Socket, J161 Conn_01x02_Socket, J162 Conn_01x02_Socket, J163 Conn_01x02_Socket, J164 Conn_01x02_Socket, J165 Conn_01x02_Socket, J166 Conn_01x02_Socket, J167 Conn_01x02_Socket, J168 Conn_01x02_Socket, J169 Conn_01x02_Socket, J17 Conn_01x02_Socket, J170 Conn_01x02_Socket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

Commit message: Update unconnected
Parts:
- moved R9 15.0 mm to (280.0, 117.0)
- moved R10 10.0 mm to (280.0, 115.0)
- moved J193 6.22 mm to (278.6, 110.4), turned to 90 degrees
Routing:
- net tNew: track 889.1 -> 998.0 mm, vias 3 -> 7
- net S2D: track 1039.7 -> 1109.0 mm, vias 3 -> 5
- net Net-(J193-CC1): track 34.3 -> 11.9 mm
- net S1Q: track 94.4 -> 116.1 mm, vias 2 -> 4
- net TABLE1: track 158.2 -> 178.3 mm
- net S2Q: track 119.2 -> 138.3 mm, vias 0 -> 2
- net CLK2: track 170.7 -> 187.2 mm, vias 4 -> 6
- net Net-(F1-Pad2): track 12.9 -> 23.6 mm
- net GND: track 104.8 -> 97.4 mm, vias 41 -> 40
- net (no net): track 0.00 -> 3.69 mm
- net VCC: track 141.6 -> 144.3 mm, vias 41 -> 43
- net Net-(J193-CC2): track 12.3 -> 12.5 mm, vias 0 -> 2
Other:
- board size 277 x 132 mm -> 277 x 131 mm
- board text added: "Program by placing LEDs into the plug-in sockets and watch the heads go by and run your program!"
- board text added: "TURING PCB"

Commit message: Respond to comments
Parts:
- moved J66 241.8 mm to (256.0, 144.5)
- moved J72 241.8 mm to (260.0, 144.5)
- moved J78 241.8 mm to (264.0, 144.5)
- moved J84 241.8 mm to (268.0, 144.5)
- moved J90 241.8 mm to (272.0, 144.5)
- moved J96 241.8 mm to (276.0, 144.5)
- moved R4 210.6 mm to (62.2, 22.0), turned to 180 degrees
- moved J119 208.4 mm to (251.0, 126.0)
- moved R5 207.7 mm to (66.0, 23.0), turned to 180 degrees
- moved R6 205.8 mm to (69.0, 24.0), turned to 180 degrees
- moved R7 202.8 mm to (73.0, 25.0), turned to 180 degrees
- moved J120 201.4 mm to (276.0, 126.0)
- moved J110 193.8 mm to (272.1, 126.0)
- moved J99 192.9 mm to (243.0, 126.0)
- moved R8 188.1 mm to (76.0, 27.0), turned to 180 degrees
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Routing:
- net R/L: track 688.5 -> 1144.3 mm, vias 0 -> 22
- net tNew: track 998.0 -> 1203.8 mm, vias 7 -> 24
- net TABLE8: track 85.0 -> 290.2 mm, vias 1 -> 2
- net TABLE29: track 54.4 -> 255.2 mm, vias 1 -> 2
- net TABLE4: track 173.0 -> 363.7 mm, vias 7 -> 2
- net TABLE22: track 236.4 -> 58.5 mm, vias 1 -> 2
- net S1D: track 1017.6 -> 1185.2 mm, vias 6 -> 14
- net TABLE0: track 112.2 -> 266.6 mm, vias 3 -> 2
- net TABLE21: track 225.5 -> 76.9 mm, vias 3 -> 2
- net TABLE16: track 155.2 -> 303.0 mm, vias 6 -> 2
- net TABLE17: track 132.3 -> 277.0 mm, vias 3 -> 4
- net Net-(U41-Pad4): track 25.9 -> 168.9 mm, vias 2 -> 6
- net TABLE15: track 298.3 -> 155.6 mm, vias 1 -> 4
- net TABLE26: track 67.6 -> 172.1 mm, vias 1 -> 2
- net TABLE7: track 83.7 -> 183.6 mm, vias 1 -> 4
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- added copper zone on In1.Cu, net GND
- added copper zone on In2.Cu, net VCC
- removed copper zone on B.Cu, net GND
- removed copper zone on In4.Cu, net VCC
Other:
- board size 277 x 131 mm -> 281 x 142 mm
- copper layers 6 -> 4
- board text added: "20 10"
- board text added: "21 11"
- board text added: "22 12"
- board text added: "23 13"
- board text added: "24 14"
- board text added: "25 15"
- board text added: "26 16"
- board text added: "27 17"
- board text added: "28 18"
- board text added: "29 19"
- board text added: "By Carter Pfaff"
- board text added: "How to program: 1. Look at the labeled table/operation commands 2. Plug in diodes to encode the transition table you intend 3. Run it and see what it does!"
- board text added: "Table 0"
- board text added: "Table 1"
- board text added: "Table 2"
- board text added: "Table 3"
- board text added: "Table 30"
- board text added: "Table 31"
- board text added: "Table 4"
- board text added: "Table 5"
- board text added: "Table 6"
- board text added: "Table 7"
- board text added: "Table 8"
- board text added: "Table 9"
- board text added: "Turing PCB"
- board text added: "| | |"
- board text removed: "Program by placing LEDs into the plug-in sockets and watch the heads go by and run your program!"
- board text removed: "TURING PCB"
